Commit message: add mujoco benchmark

File: python/spear/urdf/double_pendulum.urdf (robot description, URDF)
Before this commit: robot benchmark_torque_revolute, 2 links, 1 joints
Links:
- added link link_1, mass 1; visual box size=1 1 1
- link link_0: geometry visual box size=0.4 0.4 2
Joints:
- added joint joint_1: type continuous, parent link_0, child link_1, origin xyz=0 0 -0.5 rpy=0 0 0, axis 1 0 0, limit lower=-1.57 upper=1.57 effort=1000.0 velocity=0.1
- joint joint_0: origin xyz=0.6 0 0 rpy=0 0 0 -> xyz=1.2 0 0 rpy=0 0 0
