Commit message: add new pendulum.urdf and change existing pendulum.urdf -> horizontal_pendulum.urdf

File: python/spear/urdf/horizontal_pendulum.urdf (robot description, URDF)
Before this commit: robot pendulum, 3 links, 2 joints
Links:
- added link link_2, mass 0.1; collision box size=1 0.41 0.41; visual box size=1 0.41 0.41
- added link link_3, mass 0.1; collision box size=1 0.41 0.41; visual box size=1 0.41 0.41
- link base_link: geometry collision box size=1 1 1; visual box size=1 1 1
Joints:
- added joint joint_2: type fixed, parent link_1, child link_2, origin xyz=1 0 0 rpy=0 0 0, axis 0 1 0, limit lower=-0.78 upper=0.78 effort=0.0 velocity=0.0
- added joint joint_3: type fixed, parent link_2, child link_3, origin xyz=1 0 0 rpy=0 0 0, axis 0 1 0, limit lower=-0.78 upper=0.78 effort=0.0 velocity=0.0
- joint joint_0: axis 0 0 1 -> 1 0 0; origin xyz=0 0 -0.8 rpy=0 -1.57 0 -> xyz=0.5 0 0 rpy=0 0 0
- joint joint_1: origin xyz=0.8 0 0 rpy=0 0 0 -> xyz=1 0 0 rpy=0 0 0
