Commit message: fix typos

File: python/spear/urdf/fetch.urdf (robot description, URDF)
Before this commit: robot fetch, 23 links, 22 joints
Joints:
- joint arm_joint_1: limit lower=-1.221 upper=1.518 effort=131.76 velocity=1.454 -> lower=-1.518 upper=1.518 effort=131.76 velocity=1.454
- joint gripper_finger_joint_l: limit lower=0.0 upper=0.05 effort=60 velocity=0.05 -> lower=-0.05 upper=0.05 effort=60 velocity=0.05
- joint gripper_finger_joint_r: limit lower=0.0 upper=0.05 effort=60 velocity=0.05 -> lower=-0.05 upper=0.05 effort=60 velocity=0.05
- joint head_tilt_joint: limit lower=-0.76 upper=1.45 effort=0.68 velocity=1.57 -> lower=-1.45 upper=1.45 effort=0.68 velocity=1.57
- joint torso_joint: limit lower=0 upper=0.38615 effort=450.0 velocity=0.1 -> lower=0 upper=0.38615 effort=450 velocity=0.1

Commit message: fix typos, check in fetch content

File: python/spear/urdf/fetch.urdf (robot description, URDF)
Before this commit: robot fetch, 23 links, 22 joints
Links:
- link arm_link_0: geometry collision mesh filename=StaticMesh'/UrdfRobot/Fetch_V1/Meshes/arm_link_0.arm_link_0'; visual mesh filename=StaticMesh'/UrdfRobot/Fetch_V1/Meshes/arm_link_0.arm_link_0'
- link arm_link_1: geometry collision mesh filename=StaticMesh'/UrdfRobot/Fetch_V1/Meshes/arm_link_1.arm_link_1'; visual mesh filename=StaticMesh'/UrdfRobot/Fetch_V1/Meshes/arm_link_1.arm_link_1'
- link arm_link_2: geometry collision mesh filename=StaticMesh'/UrdfRobot/Fetch_V1/Meshes/arm_link_2.arm_link_2'; visual mesh filename=StaticMesh'/UrdfRobot/Fetch_V1/Meshes/arm_link_2.arm_link_2'
- link arm_link_3: geometry collision mesh filename=StaticMesh'/UrdfRobot/Fetch_V1/Meshes/arm_link_3.arm_link_3'; visual mesh filename=StaticMesh'/UrdfRobot/Fetch_V1/Meshes/arm_link_3.arm_link_3'
- link arm_link_4: geometry collision mesh filename=StaticMesh'/UrdfRobot/Fetch_V1/Meshes/arm_link_4.arm_link_4'; visual mesh filename=StaticMesh'/UrdfRobot/Fetch_V1/Meshes/arm_link_4.arm_link_4'
- link arm_link_5: geometry collision mesh filename=StaticMesh'/UrdfRobot/Fetch_V1/Meshes/arm_link_5.arm_link_5'; visual mesh filename=StaticMesh'/UrdfRobot/Fetch_V1/Meshes/arm_link_5.arm_link_5'
- link arm_link_6: geometry collision mesh filename=StaticMesh'/UrdfRobot/Fetch_V1/Meshes/arm_link_6.arm_link_6'; visual mesh filename=StaticMesh'/UrdfRobot/Fetch_V1/Meshes/arm_link_6.arm_link_6'
- link base_link: geometry collision mesh filename=StaticMesh'/UrdfRobot/Fetch_V1/Meshes/base_link.base_link'; visual mesh filename=StaticMesh'/UrdfRobot/Fetch_V1/Meshes/base_link.base_link'
- link estop_link: geometry collision mesh filename=StaticMesh'/UrdfRobot/Fetch_V1/Meshes/estop_link.estop_link'; visual mesh filename=StaticMesh'/UrdfRobot/Fetch_V1/Meshes/estop_link.estop_link'
- link gripper_finger_link_l: geometry collision mesh filename=StaticMesh'/UrdfRobot/Fetch_V1/Meshes/gripper_finger_link_l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; visual mesh filename=StaticMesh'/UrdfRobot/Fetch_V1/Meshes/gripper_finger_link_l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
- link gripper_finger_link_r: geometry collision mesh filename=StaticMesh'/UrdfRobot/Fetch_V1/Meshes/gripper_finger_link_r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; visual mesh filename=StaticMesh'/UrdfRobot/Fetch_V1/Meshes/gripper_finger_link_r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
- link gripper_link: geometry collision mesh filename=StaticMesh'/UrdfRobot/Fetch_V1/Meshes/gripper_link.gripper_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; visual mesh filename=StaticMesh'/UrdfRobot/Fetch_V1/Meshes/gripper_link.gripper_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
- link head_pan_link: geometry collision mesh filename=StaticMesh'/UrdfRobot/Fetch_V1/Meshes/head_pan_link_collisi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; visual mesh filename=StaticMesh'/UrdfRobot/Fetch_V1/Meshes/head_pan_link.head_pa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
- link head_tilt_link: geometry collision mesh filename=StaticMesh'/UrdfRobot/Fetch_V1/Meshes/head_tilt_link_collis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; visual mesh filename=StaticMesh'/UrdfRobot/Fetch_V1/Meshes/head_tilt_link.head_t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
- link laser_link: geometry collision mesh filename=StaticMesh'/UrdfRobot/Fetch_V1/Meshes/laser_link.laser_link'; visual mesh filename=StaticMesh'/UrdfRobot/Fetch_V1/Meshes/laser_link.laser_link'
- link torso_fixed_link: geometry collision mesh filename=StaticMesh'/UrdfRobot/Fetch_V1/Meshes/torso_fixed_link.tors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; visual mesh filename=StaticMesh'/UrdfRobot/Fetch_V1/Meshes/torso_fixed_link.tors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
- link torso_link: geometry collision mesh filename=StaticMesh'/UrdfRobot/Fetch_V1/Meshes/torso_link.torso_link'; visual mesh filename=StaticMesh'/UrdfRobot/Fetch_V1/Meshes/torso_link.torso_link'
- link wheel_link_l: geometry collision mesh filename=StaticMesh'/UrdfRobot/Fetch_V1/Meshes/wheel_link_l.wheel_li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; visual mesh filename=StaticMesh'/UrdfRobot/Fetch_V1/Meshes/wheel_link_l.wheel_li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
- link wheel_link_r: geometry collision mesh filename=StaticMesh'/UrdfRobot/Fetch_V1/Meshes/wheel_link_r.wheel_li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; visual mesh filename=StaticMesh'/UrdfRobot/Fetch_V1/Meshes/wheel_link_r.wheel_li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

Commit message: updated assets

File: python/spear/urdf/fetch.urdf (robot description, URDF)
Before this commit: robot fetch, 23 links, 22 joints
Links:
- link arm_link_0: geometry collision mesh filename=/UrdfRobot/Fetch_V1/Meshes/arm_link_0.arm_link_0'; visual mesh filename=/UrdfRobot/Fetch_V1/Meshes/arm_link_0.arm_link_0'
- link arm_link_1: geometry collision mesh filename=/UrdfRobot/Fetch_V1/Meshes/arm_link_1.arm_link_1'; visual mesh filename=/UrdfRobot/Fetch_V1/Meshes/arm_link_1.arm_link_1'
- link arm_link_2: geometry collision mesh filename=/UrdfRobot/Fetch_V1/Meshes/arm_link_2.arm_link_2'; visual mesh filename=/UrdfRobot/Fetch_V1/Meshes/arm_link_2.arm_link_2'
- link arm_link_3: geometry collision mesh filename=/UrdfRobot/Fetch_V1/Meshes/arm_link_3.arm_link_3'; visual mesh filename=/UrdfRobot/Fetch_V1/Meshes/arm_link_3.arm_link_3'
- link arm_link_4: geometry collision mesh filename=/UrdfRobot/Fetch_V1/Meshes/arm_link_4.arm_link_4'; visual mesh filename=/UrdfRobot/Fetch_V1/Meshes/arm_link_4.arm_link_4'
- link arm_link_5: geometry collision mesh filename=/UrdfRobot/Fetch_V1/Meshes/arm_link_5.arm_link_5'; visual mesh filename=/UrdfRobot/Fetch_V1/Meshes/arm_link_5.arm_link_5'
- link arm_link_6: geometry collision mesh filename=/UrdfRobot/Fetch_V1/Meshes/arm_link_6.arm_link_6'; visual mesh filename=/UrdfRobot/Fetch_V1/Meshes/arm_link_6.arm_link_6'
- link base_link: geometry collision mesh filename=/UrdfRobot/Fetch_V1/Meshes/base_link.base_link'; visual mesh filename=/UrdfRobot/Fetch_V1/Meshes/base_link.base_link'
- link estop_link: geometry collision mesh filename=/UrdfRobot/Fetch_V1/Meshes/estop_link.estop_link'; visual mesh filename=/UrdfRobot/Fetch_V1/Meshes/estop_link.estop_link'
- link gripper_finger_link_l: geometry collision mesh filename=/UrdfRobot/Fetch_V1/Meshes/gripper_finger_link_l.gripper_fi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; visual mesh filename=/UrdfRobot/Fetch_V1/Meshes/gripper_finger_link_l.gripper_fi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
- link gripper_finger_link_r: geometry collision mesh filename=/UrdfRobot/Fetch_V1/Meshes/gripper_finger_link_r.gripper_fi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; visual mesh filename=/UrdfRobot/Fetch_V1/Meshes/gripper_finger_link_r.gripper_fi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
- link gripper_link: geometry collision mesh filename=/UrdfRobot/Fetch_V1/Meshes/gripper_link.gripper_link'; visual mesh filename=/UrdfRobot/Fetch_V1/Meshes/gripper_link.gripper_link'
- link head_pan_link: geometry collision mesh filename=/UrdfRobot/Fetch_V1/Meshes/head_pan_link_collision.head_pan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; visual mesh filename=/UrdfRobot/Fetch_V1/Meshes/head_pan_link.head_pan_link'
- link head_tilt_link: geometry collision mesh filename=/UrdfRobot/Fetch_V1/Meshes/head_tilt_link_collision.head_ti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; visual mesh filename=/UrdfRobot/Fetch_V1/Meshes/head_tilt_link.head_tilt_link'
- link laser_link: geometry collision mesh filename=/UrdfRobot/Fetch_V1/Meshes/laser_link.laser_link'; visual mesh filename=/UrdfRobot/Fetch_V1/Meshes/laser_link.laser_link'
- link torso_fixed_link: geometry collision mesh filename=/UrdfRobot/Fetch_V1/Meshes/torso_fixed_link.torso_fixed_lin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; visual mesh filename=/UrdfRobot/Fetch_V1/Meshes/torso_fixed_link.torso_fixed_lin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
- link torso_link: geometry collision mesh filename=/UrdfRobot/Fetch_V1/Meshes/torso_link.torso_link'; visual mesh filename=/UrdfRobot/Fetch_V1/Meshes/torso_link.torso_link'
- link wheel_link_l: geometry collision mesh filename=/UrdfRobot/Fetch_V1/Meshes/wheel_link_l.wheel_link_l'; visual mesh filename=/UrdfRobot/Fetch_V1/Meshes/wheel_link_l.wheel_link_l'
- link wheel_link_r: geometry collision mesh filename=/UrdfRobot/Fetch_V1/Meshes/wheel_link_r.wheel_link_r'; visual mesh filename=/UrdfRobot/Fetch_V1/Meshes/wheel_link_r.wheel_link_r'

Commit message: can successfully load fetch but simulate physics is currently disabled

File: python/spear/urdf/fetch.urdf (robot description, URDF)
Before this commit: robot fetch, 23 links, 22 joints
Links:
- link arm_link_0: geometry collision mesh filename=/UrdfRobot/Fetch_V1/Meshes/arm_link_0.arm_link_0; visual mesh filename=/UrdfRobot/Fetch_V1/Meshes/arm_link_0.arm_link_0
- link arm_link_1: geometry collision mesh filename=/UrdfRobot/Fetch_V1/Meshes/arm_link_1.arm_link_1; visual mesh filename=/UrdfRobot/Fetch_V1/Meshes/arm_link_1.arm_link_1
- link arm_link_2: geometry collision mesh filename=/UrdfRobot/Fetch_V1/Meshes/arm_link_2.arm_link_2; visual mesh filename=/UrdfRobot/Fetch_V1/Meshes/arm_link_2.arm_link_2
- link arm_link_3: geometry collision mesh filename=/UrdfRobot/Fetch_V1/Meshes/arm_link_3.arm_link_3; visual mesh filename=/UrdfRobot/Fetch_V1/Meshes/arm_link_3.arm_link_3
- link arm_link_4: geometry collision mesh filename=/UrdfRobot/Fetch_V1/Meshes/arm_link_4.arm_link_4; visual mesh filename=/UrdfRobot/Fetch_V1/Meshes/arm_link_4.arm_link_4
- link arm_link_5: geometry collision mesh filename=/UrdfRobot/Fetch_V1/Meshes/arm_link_5.arm_link_5; visual mesh filename=/UrdfRobot/Fetch_V1/Meshes/arm_link_5.arm_link_5
- link arm_link_6: geometry collision mesh filename=/UrdfRobot/Fetch_V1/Meshes/arm_link_6.arm_link_6; visual mesh filename=/UrdfRobot/Fetch_V1/Meshes/arm_link_6.arm_link_6
- link base_link: geometry collision mesh filename=/UrdfRobot/Fetch_V1/Meshes/base_link.base_link; visual mesh filename=/UrdfRobot/Fetch_V1/Meshes/base_link.base_link
- link estop_link: geometry collision mesh filename=/UrdfRobot/Fetch_V1/Meshes/estop_link.estop_link; visual mesh filename=/UrdfRobot/Fetch_V1/Meshes/estop_link.estop_link
- link gripper_link: geometry collision mesh filename=/UrdfRobot/Fetch_V1/Meshes/gripper_link.gripper_link; visual mesh filename=/UrdfRobot/Fetch_V1/Meshes/gripper_link.gripper_link
- link head_pan_link: geometry collision mesh filename=/UrdfRobot/Fetch_V1/Meshes/head_pan_link_collision.head_pan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; visual mesh filename=/UrdfRobot/Fetch_V1/Meshes/head_pan_link.head_pan_link
- link head_tilt_link: geometry collision mesh filename=/UrdfRobot/Fetch_V1/Meshes/head_tilt_link_collision.head_ti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; visual mesh filename=/UrdfRobot/Fetch_V1/Meshes/head_tilt_link.head_tilt_link
- link laser_link: geometry collision mesh filename=/UrdfRobot/Fetch_V1/Meshes/laser_link.laser_link; visual mesh filename=/UrdfRobot/Fetch_V1/Meshes/laser_link.laser_link
- link torso_fixed_link: geometry collision mesh filename=/UrdfRobot/Fetch_V1/Meshes/torso_fixed_link.torso_fixed_link; visual mesh filename=/UrdfRobot/Fetch_V1/Meshes/torso_fixed_link.torso_fixed_link
- link torso_link: geometry collision mesh filename=/UrdfRobot/Fetch_V1/Meshes/torso_link.torso_link; visual mesh filename=/UrdfRobot/Fetch_V1/Meshes/torso_link.torso_link
- link wheel_link_l: geometry collision mesh filename=/UrdfRobot/Fetch_V1/Meshes/wheel_link_l.wheel_link_l; visual mesh filename=/UrdfRobot/Fetch_V1/Meshes/wheel_link_l.wheel_link_l
- link wheel_link_r: geometry collision mesh filename=/UrdfRobot/Fetch_V1/Meshes/wheel_link_r.wheel_link_r; visual mesh filename=/UrdfRobot/Fetch_V1/Meshes/wheel_link_r.wheel_link_r

Commit message: updated URDF functionality

File: python/spear/urdf/fetch.urdf (robot description, URDF)
Before this commit: robot fetch, 23 links, 22 joints
Links:
- link gripper_finger_link_l: mass 0.0785086 -> 0.00785086
- link gripper_finger_link_r: mass 0.0744093 -> 0.00744093
- link gripper_link: mass 1.12951 -> 0.012951
Joints:
- joint arm_joint_0: limit lower=-1.6056 upper=1.6056 effort=33.82 velocity=1.256 -> lower=-1.6056 upper=1.6056 effort=0 velocity=1.256
- joint arm_joint_1: limit lower=-1.518 upper=1.518 effort=131.76 velocity=1.454 -> lower=-1.518 upper=1.518 effort=0 velocity=1.454
- joint arm_joint_2: limit effort=76.94 velocity=1.571 -> effort=0 velocity=1.571
- joint arm_joint_3: limit lower=-2.251 upper=2.251 effort=66.18 velocity=1.521 -> lower=-2.251 upper=2.251 effort=0 velocity=1.521
- joint arm_joint_4: limit effort=29.35 velocity=1.571 -> effort=0 velocity=1.571
- joint arm_joint_5: limit lower=-2.16 upper=2.16 effort=25.7 velocity=2.268 -> lower=-2.16 upper=2.16 effort=0 velocity=2.268
- joint arm_joint_6: limit effort=7.36 velocity=2.268 -> effort=0 velocity=2.268
- joint gripper_finger_joint_l: limit lower=-0.05 upper=0.05 effort=60 velocity=0.05 -> lower=-0.025 upper=0.025 effort=0 velocity=0.05
- joint gripper_finger_joint_r: limit lower=-0.05 upper=0.05 effort=60 velocity=0.05 -> lower=-0.025 upper=0.025 effort=0 velocity=0.05
- joint torso_joint: limit lower=0 upper=0.38615 effort=450 velocity=0.1 -> (none)

File: python/spear/urdf/pendulum.urdf (robot description, URDF)
Before this commit: robot pendulum, 3 links, 2 joints
Links:
- added link link_2, mass 0.1; collision box size=1 0.41 0.41; visual box size=1 0.41 0.41
- added link link_3, mass 0.1; collision box size=1 0.41 0.41; visual box size=1 0.41 0.41
- link base_link: mass 0.1 -> 100.0
Joints:
- added joint joint_2: type fixed, parent link_1, child link_2, origin xyz=1 0 0 rpy=0 0 0, axis 0 1 0, limit lower=-0.78 upper=0.78 effort=0.0 velocity=0.0
- added joint joint_3: type fixed, parent link_2, child link_3, origin xyz=1 0 0 rpy=0 0 0, axis 0 1 0, limit lower=-0.78 upper=0.78 effort=0.0 velocity=0.0
- joint joint_0: origin xyz=1 0 0 rpy=0 0 0 -> xyz=0.5 0 0 rpy=0 0 0
- joint joint_1: type continuous -> fixed

Commit message: Didn't add DebugWidget to apartment_0000.
"cleaned up assets in unreal_plugins and debug_0000 to better match
latest content guidelines, added ModelingToolsEditorMode to uproject
because it is helpful for debugging and cleanup, added DebugWidget to
apartment_0000"

File: python/spear/urdf/fetch.urdf (robot description, URDF)
Before this commit: robot fetch, 23 links, 22 joints
Links:
- link arm_link_0: geometry collision mesh filename=/UrdfRobot/Fetch_V1/Meshes/SM_arm_link_0.SM_arm_link_0; visual mesh filename=/UrdfRobot/Fetch_V1/Meshes/SM_arm_link_0.SM_arm_link_0
- link arm_link_1: geometry collision mesh filename=/UrdfRobot/Fetch_V1/Meshes/SM_arm_link_1.SM_arm_link_1; visual mesh filename=/UrdfRobot/Fetch_V1/Meshes/SM_arm_link_1.SM_arm_link_1
- link arm_link_2: geometry collision mesh filename=/UrdfRobot/Fetch_V1/Meshes/SM_arm_link_2.SM_arm_link_2; visual mesh filename=/UrdfRobot/Fetch_V1/Meshes/arm_link_2.arm_link_2
- link arm_link_3: geometry collision mesh filename=/UrdfRobot/Fetch_V1/Meshes/SM_arm_link_3.SM_arm_link_3; visual mesh filename=/UrdfRobot/Fetch_V1/Meshes/SM_arm_link_3.SM_arm_link_3
- link arm_link_4: geometry collision mesh filename=/UrdfRobot/Fetch_V1/Meshes/SM_arm_link_4.SM_arm_link_4; visual mesh filename=/UrdfRobot/Fetch_V1/Meshes/SM_arm_link_4.SM_arm_link_4
- link arm_link_5: geometry collision mesh filename=/UrdfRobot/Fetch_V1/Meshes/SM_arm_link_5.SM_arm_link_5; visual mesh filename=/UrdfRobot/Fetch_V1/Meshes/SM_arm_link_5.SM_arm_link_5
- link arm_link_6: geometry collision mesh filename=/UrdfRobot/Fetch_V1/Meshes/SM_arm_link_6.SM_arm_link_6; visual mesh filename=/UrdfRobot/Fetch_V1/Meshes/SM_arm_link_6.SM_arm_link_6
- link base_link: geometry collision mesh filename=/UrdfRobot/Fetch_V1/Meshes/SM_base_link.SM_base_link; visual mesh filename=/UrdfRobot/Fetch_V1/Meshes/SM_base_link.SM_base_link
- link estop_link: geometry collision mesh filename=/UrdfRobot/Fetch_V1/Meshes/SM_estop_link.SM_estop_link; visual mesh filename=/UrdfRobot/Fetch_V1/Meshes/SM_estop_link.SM_estop_link
- link gripper_finger_link_l: geometry collision mesh filename=/UrdfRobot/Fetch_V1/Meshes/SM_gripper_finger_link_l.SM_grip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; visual mesh filename=/UrdfRobot/Fetch_V1/Meshes/SM_gripper_finger_link_l.SM_grip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
- link gripper_finger_link_r: geometry collision mesh filename=/UrdfRobot/Fetch_V1/Meshes/SM_gripper_finger_link_r.SM_grip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; visual mesh filename=/UrdfRobot/Fetch_V1/Meshes/SM_gripper_finger_link_r.SM_grip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
- link gripper_link: geometry collision mesh filename=/UrdfRobot/Fetch_V1/Meshes/SM_gripper_link.SM_gripper_link; visual mesh filename=/UrdfRobot/Fetch_V1/Meshes/SM_gripper_link.SM_gripper_link
- link head_pan_link: geometry collision mesh filename=/UrdfRobot/Fetch_V1/Meshes/SM_head_pan_link_collision.SM_he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; visual mesh filename=/UrdfRobot/Fetch_V1/Meshes/head_pan_link.head_pan_link
- link head_tilt_link: geometry collision mesh filename=/UrdfRobot/Fetch_V1/Meshes/SM_head_tilt_link_collision.SM_h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; visual mesh filename=/UrdfRobot/Fetch_V1/Meshes/SM_head_tilt_link.SM_head_tilt_l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
- link laser_link: geometry collision mesh filename=/UrdfRobot/Fetch_V1/Meshes/SM_laser_link.SM_laser_link; visual mesh filename=/UrdfRobot/Fetch_V1/Meshes/SM_laser_link.SM_laser_link
- link torso_fixed_link: geometry collision mesh filename=/UrdfRobot/Fetch_V1/Meshes/SM_torso_fixed_link.SM_torso_fix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; visual mesh filename=/UrdfRobot/Fetch_V1/Meshes/SM_torso_fixed_link.SM_torso_fix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
- link torso_link: geometry collision mesh filename=/UrdfRobot/Fetch_V1/Meshes/SM_torso_link.SM_torso_link; visual mesh filename=/UrdfRobot/Fetch_V1/Meshes/SM_torso_link.SM_torso_link
- link wheel_link_l: geometry collision mesh filename=/UrdfRobot/Fetch_V1/Meshes/SM_wheel_link_l.SM_wheel_link_l; visual mesh filename=/UrdfRobot/Fetch_V1/Meshes/SM_wheel_link_l.SM_wheel_link_l
- link wheel_link_r: geometry collision mesh filename=/UrdfRobot/Fetch_V1/Meshes/SM_wheel_link_r.SM_wheel_link_r; visual mesh filename=/UrdfRobot/Fetch_V1/Meshes/SM_wheel_link_r.SM_wheel_link_r
