Commit message: support urdf fetch agent

File: python/spear/urdf/fetch_no_spear.urdf (robot description, URDF)
Before this commit: robot fetch, 23 links, 22 joints
Links:
- link caster_link_fl: geometry collision sphere radius=0.0595; visual sphere radius=0.0595
- link caster_link_fr: geometry collision sphere radius=0.0595; visual sphere radius=0.0595
- link caster_link_rl: geometry collision sphere radius=0.0595; visual sphere radius=0.0595
- link caster_link_rr: geometry collision sphere radius=0.0595; visual sphere radius=0.0595
